Commit message: New YuMi motion planning tools

File: yumi_description/urdf/yumi.urdf (robot description, URDF)
Before this commit: robot yumi, 24 links, 23 joints
Links:
- added link left_gripper_point
- added link right_suction_point
Joints:
- added joint left_gripper_joint: type fixed, parent yumi_link_7_l, child left_gripper_point, origin xyz=0 0 0.156 rpy=0 0 3.14159265359
- added joint right_suction_joint: type fixed, parent yumi_link_7_r, child right_suction_point, origin xyz=-0.001 0 0.103 rpy=0 0 3.14159265359

Commit message: Updated to new YuMi suction tip

File: yumi_description/urdf/yumi.urdf (robot description, URDF)
Before this commit: robot yumi, 26 links, 25 joints
Joints:
- joint left_gripper_joint: origin xyz=0 0 0.156 rpy=0 0 3.14159265359 -> xyz=0 0 0.188 rpy=0 0 3.14159265359

Commit message: Updated the suction tool point for the long tip

File: yumi_description/urdf/yumi.urdf (robot description, URDF)
Before this commit: robot yumi, 26 links, 25 joints
Joints:
- joint left_gripper_joint: origin xyz=0 0 0.188 rpy=0 0 3.14159265359 -> xyz=0 0 0.190 rpy=0 0 3.14159265359
